File: hardware/controller.kicad_sch (KiCad schematic)
At the start: 60 parts

Commit message: Continue schematic - finish controller and add LCD
Parts:
- added J10: Conn_01x06, symbol Connector_Generic:Conn_01x06
- added R8, R9: 1k, symbol Device:R
- gave numbers to parts that had none: 60
Connections:
- net +3V3: now also J10.2 (Pin_2)
- net +5V: now also J10.1 (Pin_1)
- net GND: now also J10.6 (Pin_6)
- net THERMISTOR_IN1: now also R8.2; no longer C7.1, J5.2 (Pin_2), R6.2
- net THERMISTOR_IN2: now also R9.2; no longer C10.1, J6.2 (Pin_2), R7.2
- net AUX1: now reaches U1.45 (PB6)
- net AUX1: now also J10.3 (Pin_3)
- net AUX2: now reaches U1.46 (PB7)
- net AUX2: now also J10.4 (Pin_4)
- net AUX3: now reaches U1.47 (PB8)
- net AUX3: now also J10.5 (Pin_5)
- new net: C7.1, J5.2 (Pin_2), R6.2, R8.1
- new net: C10.1, J6.2 (Pin_2), R7.2
- no-connect marks 7 -> 29

Commit message: Schematic nearly finished
Parts:
- removed J5: Conn_01x02, symbol Connector_Generic:Conn_01x02
- added J?: Conn_01x02, symbol Connector_Generic:Conn_01x02
Connections:
- net GND: now also C10.2, J6.1 (Pin_1)
- net at C7.1, R6.2, R8.1: now also J?.2 (Pin_2)
- net at C10.1, J6.2 (Pin_2), R7.2: now also R9.1
- no-connect marks 29 -> 31
Changed lines of the file:
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@@
   (junction (at 335.28 162.56) (diameter 0) (color 0 0 0 0)
   )
-  (junction (at 214.63 151.13) (diameter 0) (color 0 0 0 0)
-  )
   (junction (at 336.55 35.56) (diameter 0) (color 0 0 0 0)
   )
   (junction (at 368.3 30.48) (diameter 0) (color 0 0 0 0)
   )
+  (junction (at 223.5199 120.65) (diameter 0) (color 0 0 0 0)
+  )
   (junction (at 353.06 30.48) (diameter 0) (color 0 0 0 0)
   )
   (junction (at 223.52 48.26) (diameter 0) (color 0 0 0 0)
   )
-  (junction (at 214.6299 123.1435) (diameter 0) (color 0 0 0 0)
-  )
   (junction (at 365.76 104.14) (diameter 0) (color 0 0 0 0)
   )
@@
   (junction (at 367.03 157.48) (diameter 0) (color 0 0 0 0)
   )
+  (junction (at 223.52 156.21) (diameter 0) (color 0 0 0 0)
+  )
   (junction (at 351.79 157.48) (diameter 0) (color 0 0 0 0)
   )
@@
   (junction (at 351.79 149.86) (diameter 0) (color 0 0 0 0)
   )
-  (junction (at 231.14 148.59) (diameter 0) (color 0 0 0 0)
-  )
   (junction (at 367.03 149.86) (diameter 0) (color 0 0 0 0)
   )
   (junction (at 334.01 116.84) (diameter 0) (color 0 0 0 0)
   )
-  (junction (at 223.5199 120.6035) (diameter 0) (color 0 0 0 0)
-  )
   (junction (at 365.76 111.76) (diameter 0) (color 0 0 0 0)
   )
@@
   (junction (at 368.3 63.5) (diameter 0) (color 0 0 0 0)
   )
-  (junction (at 223.5199 120.65) (diameter 0) (color 0 0 0 0)
-  )
   (junction (at 223.52 92.71) (diameter 0) (color 0 0 0 0)
   )
@@
   (junction (at 368.3 22.86) (diameter 0) (color 0 0 0 0)
   )
-  (junction (at 223.5199 128.2235) (diameter 0) (color 0 0 0 0)
-  )
   (junction (at 219.71 199.39) (diameter 0) (color 0 0 0 0)
   )
@@
   (junction (at 233.68 207.01) (diameter 0) (color 0 0 0 0)
   )
-  (junction (at 223.52 156.21) (diameter 0) (color 0 0 0 0)
-  )
   (junction (at 353.06 63.5) (diameter 0) (color 0 0 0 0)
   )
+  (no_connect (at 62.23 163.83))
+  (no_connect (at 30.48 173.99))
   (no_connect (at 57.15 90.17))
   (no_connect (at 57.15 92.71))
@@
     (stroke (width 0) (type default) (color 0 0 0 0))
   )
-  (wire (pts (xy 231.1401 148.6365) (xy 223.5201 148.6365))
-    (stroke (width 0) (type default) (color 0 0 0 0))
-  )
   (polyline (pts (xy 199.39 106.68) (xy 199.39 134.62))
     (stroke (width 0) (type default) (color 0 0 0 0))
@@
     (stroke (width 0) (type default) (color 0 0 0 0))
   )
+  (wire (pts (xy 223.5199 120.65) (xy 223.52 120.65))
+    (stroke (width 0) (type default) (color 0 0 0 0))
+  )
   (polyline (pts (xy 15.24 170.18) (xy 15.24 138.43))
     (stroke (width 0) (type default) (color 0 0 0 0))
@@
     (stroke (width 0) (type default) (color 0 0 0 0))
   )
-  (wire (pts (xy 214.6301 151.1765) (xy 215.9001 151.1765))
-    (stroke (width 0) (type default) (color 0 0 0 0))
-  )
   (wire (pts (xy 246.38 78.74) (xy 246.38 67.31))
     (stroke (width 0) (type default) (color 0 0 0 0))
@@
     (stroke (width 0) (type default) (color 0 0 0 0))
   )
-  (wire (pts (xy 215.9001 151.1765) (xy 215.9001 156.2565))
-    (stroke (width 0) (type default) (color 0 0 0 0))
-  )
   (wire (pts (xy 139.7 85.09) (xy 133.35 85.09))
     (stroke (width 0) (type default) (color 0 0 0 0))
@@
     (stroke (width 0) (type default) (color 0 0 0 0))
   )
-  (wire (pts (xy 214.6299 120.6035) (xy 223.5199 120.6035))
-    (stroke (width 0) (type default) (color 0 0 0 0))
-  )
   (wire (pts (xy 217.17 48.26) (xy 217.17 45.72))
     (stroke (width 0) (type default) (color 0 0 0 0))
   )
-  (wire (pts (xy 223.52 120.65) (xy 223.5199 120.65))
+  (wire (pts (xy 214.63 120.65) (xy 223.5199 120.65))
     (stroke (width 0) (type default) (color 0 0 0 0))
   )
@@
     (stroke (width 0) (type default) (color 0 0 0 0))
   )
-  (wire (pts (xy 215.9001 156.2565) (xy 223.5201 156.2565))
-    (stroke (width 0) (type default) (color 0 0 0 0))
-  )
   (wire (pts (xy 133.35 80.01) (xy 143.51 80.01))
     (stroke (width 0) (type default) (color 0 0 0 0))
@@
     (stroke (width 0) (type default) (color 0 0 0 0))
   )
+  (wire (pts (xy 223.52 148.59) (xy 231.14 148.59))
+    (stroke (width 0) (type default) (color 0 0 0 0))
+  )
   (wire (pts (xy 116.84 177.8) (xy 127 177.8))
     (stroke (width 0) (type default) (color 0 0 0 0))
@@
     (stroke (width 0) (type default) (color 0 0 0 0))
   )
+  (wire (pts (xy 214.63 151.13) (xy 218.44 151.13))
+    (stroke (width 0) (type default) (color 0 0 0 0))
+  )
   (wire (pts (xy 374.65 22.86) (xy 368.3 22.86))
     (stroke (width 0) (type default) (color 0 0 0 0))
@@
     (stroke (width 0) (type default) (color 0 0 0 0))
   )
+  (wire (pts (xy 218.44 156.21) (xy 223.52 156.21))
+    (stroke (width 0) (type default) (color 0 0 0 0))
+  )
   (polyline (pts (xy 325.12 140.97) (xy 325.12 177.8))
     (stroke (width 0) (type default) (color 0 0 0 0))
@@
     (stroke (width 0) (type default) (color 0 0 0 0))
   )
-  (wire (pts (xy 214.63 123.19) (xy 215.9 123.19))
-    (stroke (width 0) (type default) (color 0 0 0 0))
-  )
   (wire (pts (xy 335.28 35.56) (xy 336.55 35.56))
     (stroke (width 0) (type default) (color 0 0 0 0))
@@
     (stroke (width 0) (type default) (color 0 0 0 0))
   )
+  (wire (pts (xy 218.44 151.13) (xy 218.44 156.21))
+    (stroke (width 0) (type default) (color 0 0 0 0))
+  )
   (wire (pts (xy 217.17 45.72) (xy 212.09 45.72))
     (stroke (width 0) (type default) (color 0 0 0 0))
@@
   )
   (wire (pts (xy 350.52 111.76) (xy 365.76 111.76))
-    (stroke (width 0) (type default) (color 0 0 0 0))
-  )
-  (wire (pts (xy 215.9 128.27) (xy 223.52 128.27))
-    (stroke (width 0) (type default) (color 0 0 0 0))
-  )
-  (wire (pts (xy 215.9 123.19) (xy 215.9 128.27))
     (stroke (width 0) (type default) (color 0 0 0 0))
   )
@@
     (pin "2")
   )
-  (symbol (lib_id "power:GND") (at 223.5201 156.2565 0) (unit 1)
-    (in_bom yes) (on_board yes) (fields_autoplaced)
-    (property "Reference" "#PWR017" (id 0) (at 223.5201 162.6065 0)
-      (effects (font (size 1.27 1.27)) hide)
-    )
-    (property "Value" "GND" (id 1) (at 223.5201 160.6999 0))
-    (property "Footprint" "" (id 2) (at 223.5201 156.2565 0)
-      (effects (font (size 1.27 1.27)) hide)
-    )
-    (property "Datasheet" "" (id 3) (at 223.5201 156.2565 0)
+  (symbol (lib_id "power:GND") (at 223.52 156.21 0) (unit 1)
+    (in_bom yes) (on_board yes) (fields_autoplaced)
+    (property "Reference" "#PWR017" (id 0) (at 223.52 162.56 0)
+      (effects (font (size 1.27 1.27)) hide)
+    )
+    (property "Value" "GND" (id 1) (at 223.52 160.6534 0))
+    (property "Footprint" "" (id 2) (at 223.52 156.21 0)
+      (effects (font (size 1.27 1.27)) hide)
+    )
+    (property "Datasheet" "" (id 3) (at 223.52 156.21 0)
       (effects (font (size 1.27 1.27)) hide)
     )
@@
     )
     (pin "1")
-  )
-  (symbol (lib_id "Connector_Generic:Conn_01x02") (at 209.5499 123.1435 180) (unit 1)
-    (in_bom yes) (on_board yes) (fields_autoplaced)
-    (property "Reference" "J5" (id 0) (at 209.5499 115.6337 0))
-    (property "Value" "Conn_01x02" (id 1) (at 209.5499 118.1706 0))
-    (property "Footprint" "" (id 2) (at 209.5499 123.1435 0)
-      (effects (font (size 1.27 1.27)) hide)
-    )
-    (property "Datasheet" "~" (id 3) (at 209.5499 123.1435 0)
-      (effects (font (size 1.27 1.27)) hide)
-    )
-    (pin "1")
-    (pin "2")
   )
   (symbol (lib_id "Device:C") (at 223.5199 124.4135 0) (unit 1)
@@
     (pin "3")
   )
+  (symbol (lib_id "Connector_Generic:Conn_01x02") (at 209.55 123.19 180) (unit 1)
+    (in_bom yes) (on_board yes) (fields_autoplaced)
+    (property "Reference" "J?" (id 0) (at 209.55 115.6802 0))
+    (property "Value" "Conn_01x02" (id 1) (at 209.55 118.2171 0))
+    (property "Footprint" "" (id 2) (at 209.55 123.19 0)
+      (effects (font (size 1.27 1.27)) hide)
+    )
+    (property "Datasheet" "~" (id 3) (at 209.55 123.19 0)
+      (effects (font (size 1.27 1.27)) hide)
+    )
+    (pin "1")
+    (pin "2")
+  )
   (symbol (lib_id "power:GND") (at 219.71 207.01 0) (unit 1)
     (in_bom yes) (on_board yes) (fields_autoplaced)
@@
     (pin "2")
   )
-  (symbol (lib_id "power:GND") (at 223.52 128.27 0) (unit 1)
-    (in_bom yes) (on_board yes) (fields_autoplaced)
-    (property "Reference" "#PWR015" (id 0) (at 223.52 134.62 0)
-      (effects (font (size 1.27 1.27)) hide)
-    )
-    (property "Value" "GND" (id 1) (at 223.52 132.7134 0))
-    (property "Footprint" "" (id 2) (at 223.52 128.27 0)
-      (effects (font (size 1.27 1.27)) hide)
-    )
-    (property "Datasheet" "" (id 3) (at 223.52 128.27 0)
-      (effects (font (size 1.27 1.27)) hide)
-    )
+  (symbol (lib_id "power:GND") (at 243.84 125.73 0) (unit 1)
+    (in_bom yes) (on_board yes) (fields_autoplaced)
+    (property "Reference" "#PWR015" (id 0) (at 243.84 132.08 0)
+      (effects (font (size 1.27 1.27)) hide)
+    )
+    (property "Value" "GND" (id 1) (at 243.84 130.1734 0))
+    (property "Footprint" "" (id 2) (at 243.84 125.73 0)
+      (effects (font (size 1.27 1.27)) hide)
+    )
+    (property "Datasheet" "" (id 3) (at 243.84 125.73 0)
+      (effects (font (size 1.27 1.27)) hide)
+    )

Commit message: Update schematic and part assignment
Parts:
- removed J6, J?: Conn_01x02, symbol Connector_Generic:Conn_01x02
- added C31, C32, C33, C34, C? (x2): 100nF, Capacitor_SMD:C_0402_1005Metric, symbol Device:C
- added D?: D, Diode_THT:D_DO-201AD_P12.70mm_Horizontal, symbol Device:D
- added D?: D_TVS_5V, Diode_SMD:D_SMA_Handsoldering, symbol Device:D_TVS
- added J16: Conn_01x02 Screw, symbol Connector_Generic:Conn_01x02
- added J? (x2): Conn_01x03, symbol Connector_Generic:Conn_01x03
- added J?: Conn_01x02, symbol Connector_Generic:Conn_01x02
- added JP2, JP?: Jumper_3_Bridged12, Connector_PinHeader_2.54mm:PinHeader_1x03_P2.54mm_Vertical, symbol Jumper:Jumper_3_Bridged12
- added Q?: AO3400A, Package_TO_SOT_SMD:SOT-23, symbol Transistor_FET:AO3400A
- added R40, R41: 10k 0603, Resistor_SMD:R_0603_1608Metric_Pad0.98x0.95mm_HandSolder, symbol Device:R
- added R42, R43: 2.2, Resistor_SMD:R_0603_1608Metric_Pad0.98x0.95mm_HandSolder, symbol Device:R
- added R?: 100, Resistor_SMD:R_0402_1005Metric, symbol Device:R
- added R?: 10k, Resistor_SMD:R_0402_1005Metric, symbol Device:R
- BZ1: footprint (none) -> Homebrew:MURATA_PKM13EPYH4000-A0; MPN (none) -> PKM13EPYH4000-A0
- C1, C10, C12, C13, C2, C3, C7: footprint (none) -> Capacitor_SMD:C_0402_1005Metric; LCSC (none) -> C52923
- C11, C5, C6: footprint (none) -> Capacitor_SMD:C_0402_1005Metric; LCSC (none) -> C307331
- C4: footprint (none) -> Capacitor_SMD:C_0603_1608Metric; LCSC (none) -> C96446
- C8, C9: footprint (none) -> Capacitor_SMD:C_0402_1005Metric; LCSC (none) -> C15195
- D1: footprint (none) -> LED_SMD:LED_0805_2012Metric; LCSC (none) -> C84256
- D2: footprint (none) -> Diode_SMD:D_SMA_Handsoldering; MPN (none) -> 824501131
- D3, D4, D5: footprint (none) -> Diode_SMD:D_SMA_Handsoldering; MPN (none) -> 824501600
- D6, D7, D8, D9: footprint (none) -> Diode_THT:D_DO-201AD_P12.70mm_Horizontal; MPN (none) -> SB10150TA
- J1: footprint (none) -> Homebrew:FRAMATOME_10118194-0001LF_fixed_bridges; LCSC (none) -> C132563
- J10: value Conn_01x06 -> Conn_01x06 Header
- J2: value Conn_01x04 -> Conn_01x04 Header
- JP1: footprint (none) -> Connector_PinHeader_2.54mm:PinHeader_1x03_P2.54mm_Vertical
- Q1, Q2, Q3, Q4: LCSC (none) -> C20917
- R1, R18, R19: footprint (none) -> Resistor_SMD:R_0402_1005Metric; LCSC (none) -> C11702
- R10, R11, R12, R13: footprint (none) -> Resistor_SMD:R_0402_1005Metric; LCSC (none) -> C25744
- R14, R15, R16, R17: footprint (none) -> Resistor_SMD:R_0402_1005Metric; LCSC (none) -> C25076
- R2: value 3k3 -> 4k7; footprint (none) -> Resistor_SMD:R_0402_1005Metric; LCSC (none) -> C25900
- R3, R4: footprint (none) -> Resistor_SMD:R_0603_1608Metric; LCSC (none) -> C25190
- R5: value 47 -> 27; footprint (none) -> Resistor_SMD:R_0603_1608Metric; LCSC (none) -> C25190
- R6, R7: value 4k7 -> 4k7 0603; footprint (none) -> Resistor_SMD:R_0603_1608Metric_Pad0.98x0.95mm_HandSolder; LCSC (none) -> C23162
- R8, R9: value 1k -> 1k 0603; footprint (none) -> Resistor_SMD:R_0603_1608Metric_Pad0.98x0.95mm_HandSolder; LCSC (none) -> C21190
- SW1: footprint (none) -> Homebrew:SW_TACTILE_5.1MM_TS-1187A-C-D-B; LCSC (none) -> C318884
- U1: LCSC (none) -> C529329
- U2: LCSC (none) -> C84681
Connections:
- net +12V: now also J16.1 (Pin_1), JP2.3 (B), JP?.3 (B); no longer D2.2 (A2), D6.1 (K), J11.1 (Pin_1)
- net +3V3: now also J?.3 (Pin_3), J?.3 (Pin_3)
- net +5V: now also JP2.1 (A), JP?.1 (A), R40.2, R41.2, R42.1, R43.1; no longer J8.1 (Pin_1), J9.1 (Pin_1)
- net FAN_OUT: now also C31.1
- net GND: now also C7.2, C31.2, C32.2, C33.2, C34.2, C?.2, C?.2, J16.2 (Pin_2), J?.1 (Pin_1), J?.1 (Pin_1), Q?.2 (S), R?.1
- net SSR1_OUT: now also R40.1
- net SSR2_OUT: now also R41.1
- net STIR_OUT: now also C32.1
- net at C7.1, R6.2, R8.1: now also J?.2 (Pin_2)
- net at D3.2 (A2), D7.1 (K), J7.1 (Pin_1)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: now also C33.1
- net at C10.1, R7.2, R9.1: now also J?.2 (Pin_2)
- new net: C34.1, D2.2 (A2), D6.1 (K), J11.1 (Pin_1), JP2.2 (C)
- new net: Q?.1 (G), R?.2
- new net: J9.1 (Pin_1), R43.2
- new net: C?.1, D?.1 (K), D?.2 (A2), J?.1 (Pin_1), JP?.2 (C)
- new net: J8.1 (Pin_1), R42.2
- new net RELAY_EN: R?.1, R?.2
- new net RELAY_OUT: C?.1, D?.1 (A1), D?.2 (A), J?.2 (Pin_2), Q?.3 (D)
Other:
- note added: "12V AUX OUT"
- moved on the sheet: D3, D4, D5, D7, D8, D9, J10, J7, J8, J9, JP1, Q2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

Commit message: Finish assigning footprints
Parts:
- removed J16: Conn_01x02 Screw, symbol Connector_Generic:Conn_01x02
- removed J7, J8, J9, J?: Conn_01x02, symbol Connector_Generic:Conn_01x02
- added J? (x5): Conn_01x03 MiniPV, Homebrew:MiniPV_69167-X03XXX_1x03_P2.54mm_Polarized_Vertical, symbol Connector_Generic:Conn_01x03
- J10: footprint (none) -> Connector_PinHeader_2.54mm:PinHeader_1x06_P2.54mm_Vertical
- J11: value Conn_01x04 -> Conn_01x04 MiniPV; footprint (none) -> Connector_PinHeader_2.54mm:PinHeader_1x04_P2.54mm_Vertical
- J2: footprint (none) -> Connector_PinHeader_2.54mm:PinHeader_1x04_P2.54mm_Vertical
- J3, J4: value Conn_01x02 -> Conn_01x02 MiniPV; footprint (none) -> Homebrew:MiniPV_76384-X02XX_1x02_P2.54mm_Vertical
- J? (x2): value Conn_01x03 -> Conn_01x03 MiniPV; footprint (none) -> Homebrew:MiniPV_69167-X03XXX_1x03_P2.54mm_Polarized_Vertical
Connections:
- net +12V: now also J?.2 (Pin_2)
- net GND: now also J?.1 (Pin_1)
- net RELAY_OUT: now also J?.1 (Pin_1)
- net SSR1_OUT: now also J?.1 (Pin_1)
- net SSR2_OUT: now also J?.1 (Pin_1)
- net STIR_OUT: now also J?.1 (Pin_1)
- net at C33.1, D3.2 (A2), D7.1 (K)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: now also J?.2 (Pin_2)
- net at R43.2: now also J?.2 (Pin_2)
- net at C?.1, D?.1 (K), D?.2 (A2)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: now also J?.2 (Pin_2)
- net at R42.2: now also J?.2 (Pin_2)
- no-connect marks 31 -> 36
Other:
- moved on the sheet: C?, D?, JP?, Q?, R?

Commit message: Start layout
Parts:
- D13: renamed from D?; footprint Diode_THT:D_DO-201AD_P12.70mm_Horizontal -> Diode_SMD:D_SMA; LCSC (none) -> C8678; MPN SB10150TA -> (none)
- D6, D7, D8, D9: footprint Diode_THT:D_DO-201AD_P12.70mm_Horizontal -> Diode_SMD:D_SMA; LCSC (none) -> C8678; MPN SB10150TA -> (none)
- gave numbers to parts that had none: 14
