File: hardware/controller.kicad_sch (KiCad schematic)
At the start: 79 parts, among them J10 Conn_01x06 Header, J11 Conn_01x04 MiniPV, J16 Conn_01x03 MiniPV, J2 Conn_01x04 Header, J3 Conn_01x02 MiniPV, J4 Conn_01x02 MiniPV, J5 Conn_01x03 MiniPV, J6 Conn_01x03 MiniPV, J7 Conn_01x03 MiniPV, J8 Conn_01x03 MiniPV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

Commit message: First pass at layout
Parts:
- J11: footprint Connector_PinHeader_2.54mm:PinHeader_1x04_P2.54mm_Vertical -> Homebrew:MiniPV_69167-X04XXX_1x04_P2.54mm_Polarized_Vertical
Changed lines of the file:
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@@
       (effects (font (size 1.27 1.27)) (justify left))
     )
-    (property "Footprint" "Connector_PinHeader_2.54mm:PinHeader_1x04_P2.54mm_Vertical" (id 2) (at 391.16 77.47 0)
+    (property "Footprint" "Homebrew:MiniPV_69167-X04XXX_1x04_P2.54mm_Polarized_Vertical" (id 2) (at 391.16 77.47 0)
       (effects (font (size 1.27 1.27)) hide)
     )

Commit message: Hardware revision v1.0
Parts:
- R5: LCSC C25091 -> C25092
Connections:
- net FAN_PWM_OUT: now also U1.33 (PA11)
- net FAN_TACH_IN: now also U1.39 (PD1)
- net RELAY_EN: now also U1.40 (PD2)
- no-connect marks 30 -> 27
Changed lines of the file:
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@@
   (no_connect (at 133.35 44.45))
   (no_connect (at 133.35 49.53))
-  (no_connect (at 57.15 67.31))
   (no_connect (at 57.15 105.41))
   (no_connect (at 57.15 44.45))
@@
   (no_connect (at 57.15 46.99))
   (no_connect (at 179.07 260.35))
-  (no_connect (at 133.35 57.15))
   (no_connect (at 383.54 22.86))
   (no_connect (at 379.73 163.83))
@@
   (no_connect (at 57.15 118.11))
   (no_connect (at 133.35 67.31))
-  (no_connect (at 133.35 59.69))
   (no_connect (at 57.15 69.85))
   (wire (pts (xy 219.71 207.01) (xy 231.14 207.01))
@@
     (effects (font (size 1.27 1.27)) (justify right bottom))
   )
+  (label "RELAY_EN" (at 133.35 59.69 0)
+    (effects (font (size 1.27 1.27)) (justify left bottom))
+  )
   (label "SWDIO" (at 57.15 72.39 180)
     (effects (font (size 1.27 1.27)) (justify right bottom))
@@
     (effects (font (size 1.27 1.27)) (justify right bottom))
   )
+  (label "FAN_PWM_OUT" (at 57.15 67.31 180)
+    (effects (font (size 1.27 1.27)) (justify right bottom))
+  )
   (label "SPI_NSS1" (at 256.54 46.99 0)
     (effects (font (size 1.27 1.27)) (justify left bottom))
@@
   )
   (label "AUX_EN" (at 133.35 41.91 0)
+    (effects (font (size 1.27 1.27)) (justify left bottom))
+  )
+  (label "FAN_TACH_IN" (at 133.35 57.15 0)
     (effects (font (size 1.27 1.27)) (justify left bottom))
   )
@@
       (effects (font (size 1.27 1.27)) hide)
     )
-    (property "LCSC" "C25091" (id 4) (at 214.63 199.39 0)
-      (effects (font (size 1.27 1.27)) hide)
-    )
+    (property "LCSC" "C25092" (id 4) (at 214.63 199.39 0)
+      (effects (font (size 1.27 1.27)) hide)
+    )
