File: hardware/kelvin-kontroller.kicad_pcb (KiCad board)
At the start: 2 copper layers, 140 x 80 mm, 139 parts, among them J1 USB_B_Micro, J10 Conn_01x06 Header, J11 Conn_01x04 MiniPV, J12 USB_B_Micro, J13 Conn_01x04 Header, J14 Conn_01x02 Terminals, J15 Conn_01x07 Header, J16 Conn_01x03 MiniPV, J17 Conn_01x03 MiniPV, J2 Conn_01x04 Header, J3 Conn_01x02 MiniPV, J4 Conn_01x02 MiniPV, J5 Conn_01x03 MiniPV, J6 Conn_01x03 MiniPV, J7 Conn_01x03 MiniPV, J8 Conn_01x03 MiniPV, J9 Conn_01x03 MiniPV, Q1 AO3400A, Q2 AO3400A, Q3 AO3400A, Q4 AO3400A, Q5 Q_NPN_BEC, Q6 Q_NPN_BEC, Q7 AO3400A, SW1 SW_Push, SW2 SW_Push, SW3 RotaryEncoder_Switch, U1 STM32G030C8T6, U2 CH340C, U3 MAX31855KASA, U4 MAX31855KASA, U5 AMS1117-3.3, U6 ESP32-WROOM-32, U7 XL1509-5.0E1, U8 CH340C

Commit message: Continue layout, add SPI flash
Parts:
- removed J17: Conn_01x03 MiniPV, Homebrew:MiniPV_69167-X03XXX_1x03_P2.54mm_Polarized_Vertical
- added C37: 100nF, Capacitor_SMD:C_0402_1005Metric, F.Cu at (72.8, 63.0)
- added JP4: Jumper_3_Bridged12, Connector_PinHeader_2.54mm:PinHeader_1x03_P2.54mm_Vertical, F.Cu at (69.0, 60.8)
- added TH1: Thermistor_NTC, Capacitor_THT:C_Disc_D3.0mm_W2.0mm_P2.50mm, F.Cu at (72.9, 60.2)
- added U9: W25Q128JVSIQ, Package_SO:SOIC-8_5.275x5.275mm_P1.27mm, F.Cu at (93.3, 199.7)
- C11: value 100nF -> 1uF; moved to F.Cu
- C6: value 100nF -> 470nF
- D12: value D_TVS_5V -> D; footprint Diode_SMD:D_SMA_Handsoldering -> Diode_SMD:D_SMA
- D9: value D -> D_TVS_5V; footprint Diode_SMD:D_SMA -> Diode_SMD:D_SMA_Handsoldering
- R1: value 1k -> 470
- R17: value 100 -> 10k
- R22, R23, R24, R26, R3, R4, R5: value 27 -> 22; footprint Resistor_SMD:R_0603_1608Metric -> Resistor_SMD:R_0402_1005Metric
- R41: value 10k 0603 -> DNP 0603
- R43: value 2.2 -> 0 0603
- R44: value 10k -> 100
- R8, R9: value 1k 0603 -> 100 0603
- moved R5 273.3 mm to (199.0, 142.4), turned to 0 degrees
- moved BZ1 254.8 mm to (207.4, 142.4), turned to 0 degrees
- moved R21 253.3 mm to (143.9, 154.1), turned to 0 degrees
- moved C6 251.2 mm to (207.6, 134.9), turned to 0 degrees
- moved R1 250.7 mm to (220.5, 160.6), turned to 90 degrees
- moved R28 249.3 mm to (157.5, 154.4), turned to 90 degrees
- moved U8 243.5 mm to (156.9, 159.3), turned to 90 degrees
- moved R23 238.0 mm to (155.1, 165.5), turned to 90 degrees
- moved R30 232.6 mm to (160.6, 147.6), turned to 0 degrees
- moved D1 231.0 mm to (220.5, 157.7), turned to 90 degrees
- moved C24 224.9 mm to (162.7, 158.1), turned to -90 degrees
- moved R29 221.3 mm to (158.8, 154.4), turned to 90 degrees
- moved C25 218.4 mm to (158.6, 147.6)
- moved SW2 216.9 mm to (152.4, 144.5)
- moved Q5 216.1 mm to (160.0, 150.1), turned to 90 degrees
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Connections:
- net Net-(J12-Pad2) renamed /USB-
- net Net-(J12-Pad3) renamed /USB+
- net Net-(R22-Pad2) renamed /USB_R-
- net Net-(R23-Pad2) renamed /USB_R+
- C11 pad 1: Net-(BZ1-Pad1) -> +3V3
- C31 pad 1: /controller/FAN_OUT -> Net-(C31-Pad1)
- C31 pad 2: GND -> /controller/STIR_OUT
- C33 pad 2: GND -> /controller/RELAY_OUT
- C34 pad 2: GND -> /controller/FAN_OUT
- C35 pad 1: /controller/RELAY_OUT -> Net-(C35-Pad1)
- C35 pad 2: GND -> /controller/AUX_MOSFET_OUT
- C36 pad 1: Net-(C36-Pad1) -> /controller/RELAY_OUT
- D12 pad 1: /controller/RELAY_OUT -> Net-(C33-Pad1)
- D12 pad 2: Net-(C36-Pad1) -> /controller/RELAY_OUT
- D13 pad 1: Net-(C36-Pad1) -> Net-(C35-Pad1)
- D13 pad 2: /controller/RELAY_OUT -> /controller/AUX_MOSFET_OUT
- D3 pad 2: Net-(C33-Pad1) -> Net-(C31-Pad1)
- D5 pad 1: /controller/SSR2_OUT -> /controller/RELAY_OUT
- D5 pad 2: +5V -> Net-(C33-Pad1)
- D7 pad 1: Net-(C33-Pad1) -> Net-(C31-Pad1)
- D9 pad 1: +5V -> /controller/AUX_MOSFET_OUT
- D9 pad 2: /controller/SSR2_OUT -> Net-(C35-Pad1)
- J1 pad 2: Net-(J1-Pad2) -> /controller/USB-
- J1 pad 3: Net-(J1-Pad3) -> /controller/USB+
- J16 pad 1: /controller/SSR1_OUT -> /controller/AUX_MOSFET_OUT
- J16 pad 2: Net-(R42-Pad2) -> Net-(J16-Pad2)
- J7 pad 1: GND -> /controller/STIR_OUT
- J7 pad 2: Net-(C10-Pad1) -> Net-(C31-Pad1)
- J7 pad 3: +3V3 -> unconnected-(J7-Pad3)
- J8 pad 1: /controller/STIR_OUT -> /controller/RELAY_OUT
- J9 pad 1: /controller/RELAY_OUT -> /controller/SSR1_OUT
- J9 pad 2: Net-(C36-Pad1) -> Net-(J9-Pad2)
- JP1 pad 2: Net-(C33-Pad1) -> Net-(C31-Pad1)
- JP3 pad 2: Net-(C36-Pad1) -> Net-(C33-Pad1)
- Q4 pad 3: /controller/SSR2_OUT -> /controller/RELAY_OUT
- Q7 pad 3: /controller/RELAY_OUT -> /controller/AUX_MOSFET_OUT
- R13 pad 2: /controller/SSR2_EN -> /controller/RELAY_EN
- R17 pad 1: /controller/SSR2_EN -> GND
- R17 pad 2: Net-(Q4-Pad1) -> /controller/AUX_EN
- R3 pad 1: Net-(J1-Pad3) -> /controller/USB+
- R3 pad 2: /controller/USB+ -> /controller/USB_R+
- R4 pad 1: Net-(J1-Pad2) -> /controller/USB-
- R4 pad 2: /controller/USB- -> /controller/USB_R-
- R41 pad 1: /controller/SSR2_OUT -> /controller/AUX_MOSFET_OUT
- R41 pad 2: +5V -> Net-(C35-Pad1)
- R42 pad 2: Net-(R42-Pad2) -> Net-(J9-Pad2)
- R43 pad 1: +5V -> Net-(C35-Pad1)
- R43 pad 2: Net-(R43-Pad2) -> Net-(J16-Pad2)
- R44 pad 1: GND -> /controller/RELAY_EN
- R44 pad 2: /controller/RELAY_EN -> Net-(Q4-Pad1)
- R45 pad 1: /controller/RELAY_EN -> /controller/AUX_EN
- U1 pad 31: /controller/SSR2_EN -> /controller/AUX_EN
- U2 pad 5: /controller/USB+ -> /controller/USB_R+
- U2 pad 6: /controller/USB- -> /controller/USB_R-
- U6 pad 16: unconnected-(U6-Pad16) -> /SDA
- U6 pad 26: unconnected-(U6-Pad26) -> /SCL
- U6 pad 29: unconnected-(U6-Pad29) -> /VSPI_CS
- U6 pad 30: unconnected-(U6-Pad30) -> /VSPI_SCK
- U6 pad 31: unconnected-(U6-Pad31) -> /VSPI_MISO
- U6 pad 33: /SDA -> /VSPI_HD
- U6 pad 36: /SCL -> /VSPI_WP
- U6 pad 37: unconnected-(U6-Pad37) -> /VSPI_MOSI
Routing:
- net /USB_R-: track 0.00 -> 3.98 mm, vias 0 -> 2
- net /USB_R+: track 0.00 -> 3.60 mm, vias 0 -> 2
- net /USB-: track 0.00 -> 1.96 mm
- net /USB+: track 0.00 -> 1.96 mm
Other:
- board size 140 x 80 mm -> 116 x 72 mm

Commit message: Continue layout
Parts:
- removed C1: 1uF, Capacitor_SMD:C_0402_1005Metric
- removed C5: 100nF, Capacitor_SMD:C_0402_1005Metric
- removed J1: USB_B_Micro, Homebrew:FRAMATOME_10118194-0001LF_fixed_bridges
- removed R4: 22, Resistor_SMD:R_0402_1005Metric
- removed U2: CH340C, Package_SO:SOIC-16_3.9x9.9mm_P1.27mm
- added SW4: SW_Push, Homebrew:SW_TACTILE_5.1MM_TS-1187A-C-D-B, B.Cu at (186.3, 168.6)
- BZ1: moved to F.Cu
- C11, TH1, U9: moved to B.Cu
- R2: value 4k7 -> 10k
- R3: value 22 -> 100k
- moved R42 290.7 mm to (210.8, 115.8), turned to 90 degrees
- moved J9 274.8 mm to (208.3, 110.8), turned to -90 degrees
- moved R12 260.5 mm to (202.7, 114.9), turned to -90 degrees
- moved C3 256.8 mm to (192.4, 148.9), turned to 90 degrees
- moved C10 252.3 mm to (171.8, 156.2), turned to 0 degrees
- moved SW1 250.6 mm to (195.9, 168.7)
- moved R40 249.4 mm to (209.0, 115.8), turned to -90 degrees
- moved Q3 246.2 mm to (204.3, 112.1), turned to 0 degrees
- moved C4 245.6 mm to (193.8, 151.3), turned to -90 degrees
- moved R3 244.3 mm to (191.1, 169.1)
- moved D4 238.5 mm to (213.5, 118.6), turned to -90 degrees
- moved C2 235.8 mm to (192.4, 150.9), turned to -90 degrees
- moved U3 235.1 mm to (167.6, 134.0), turned to -90 degrees
- moved C13 234.6 mm to (163.1, 132.7), turned to -90 degrees
- moved J3 232.7 mm to (166.2, 126.1), turned to -90 degrees
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Connections:
- J2 pad 4: /controller/BOOT0_SWCLK -> /controller/SWCLK
- R2 pad 2: /controller/BOOT0 -> +3V3
- R3 pad 1: /controller/USB+ -> GND
- R3 pad 2: /controller/USB_R+ -> /controller/SWCLK
- U1 pad 13: /controller/USB_USART_TX -> unconnected-(U1-Pad13)
- U1 pad 14: /controller/USB_USART_RX -> unconnected-(U1-Pad14)
- U1 pad 36: /controller/BOOT0 -> /controller/SWCLK

Commit message: First pass at layout
Parts:
- C37, JP4: moved to B.Cu
- J11: footprint Connector_PinHeader_2.54mm:PinHeader_1x04_P2.54mm_Vertical -> Homebrew:MiniPV_69167-X04XXX_1x04_P2.54mm_Polarized_Vertical
- moved Q4 297.9 mm to (210.9, 139.6), turned to 0 degrees
- moved C35 291.7 mm to (212.0, 156.2), turned to 0 degrees
- moved R41 288.4 mm to (211.7, 158.2)
- moved J8 286.7 mm to (211.5, 130.3), turned to 90 degrees
- moved C33 274.0 mm to (213.7, 124.2), turned to -90 degrees
- moved C36 268.6 mm to (213.7, 126.1), turned to -90 degrees
- moved C32 267.3 mm to (199.7, 125.0), turned to -90 degrees
- moved J16 261.5 mm to (212.7, 148.2), turned to 90 degrees
- moved Q7 260.8 mm to (201.9, 155.2), turned to 0 degrees
- moved R13 260.7 mm to (207.4, 138.9), turned to -90 degrees
- moved R18 260.3 mm to (180.1, 134.7), turned to 90 degrees
- moved Q1 259.2 mm to (176.8, 139.3), turned to 0 degrees
- moved Q2 257.8 mm to (196.4, 138.5), turned to 0 degrees
- moved C31 257.2 mm to (199.7, 123.0), turned to -90 degrees
- moved D3 253.9 mm to (194.7, 134.8)
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Other:
- outline, holes or cut-outs redrawn

Commit message: Start routing
Parts:
- moved JP3 5.13 mm to (202.6, 132.9), turned to 0 degrees
- moved JP2 5.05 mm to (171.0, 131.4), turned to 0 degrees
- moved JP1 5.03 mm to (188.3, 131.8), turned to 0 degrees
- moved JP4 4.55 mm to (203.8, 150.1), turned to 0 degrees
- moved R20 3.09 mm to (147.0, 155.3)
- moved R21 3.09 mm to (147.0, 154.1)
Routing:
- net GND: track 0.00 -> 449.4 mm, vias 0 -> 12
- net +3V3: track 0.00 -> 216.1 mm, vias 0 -> 8
- net +5V: track 0.00 -> 197.8 mm, vias 0 -> 4
- net +12V: track 0.00 -> 170.8 mm, vias 0 -> 3
- net /ENC_BUTTON: track 0.00 -> 121.3 mm, vias 0 -> 6
- net /ENC_A: track 0.00 -> 105.6 mm, vias 0 -> 2
- net /ENC_B: track 0.00 -> 97.1 mm, vias 0 -> 2
- net /ESP_USART_RX: track 0.00 -> 75.2 mm, vias 0 -> 4
- net /ESP_USART_TX: track 0.00 -> 72.6 mm, vias 0 -> 4
- net /EN: track 0.00 -> 54.8 mm, vias 0 -> 2
- net /SDA: track 0.00 -> 42.2 mm, vias 0 -> 2
- net /SCL: track 0.00 -> 40.6 mm, vias 0 -> 2
- net /VSPI_WP: track 0.00 -> 28.3 mm, vias 0 -> 2
- net /VSPI_MISO: track 0.00 -> 25.4 mm, vias 0 -> 2
- net /IO0: track 0.00 -> 24.3 mm, vias 0 -> 2
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
Commit message: Hardware revision v1.0
Parts:
- moved R1 4.90 mm to (206.4, 169.1), turned to 180 degrees
- moved D1 2.08 mm to (203.5, 169.1), turned to 180 degrees
Connections:
- U1 pad 33: unconnected-(U1-Pad33) -> /controller/FAN_PWM_OUT
- U1 pad 39: unconnected-(U1-Pad39) -> /controller/FAN_TACH_IN
- U1 pad 40: unconnected-(U1-Pad40) -> /controller/RELAY_EN
Routing:
- net +3V3: track 216.1 -> 354.7 mm, vias 8 -> 19
- net /controller/SPI_MISO: track 0.00 -> 66.1 mm, vias 0 -> 4
- net /controller/SPI_SCK: track 0.00 -> 58.5 mm, vias 0 -> 4
- net /controller/SSR1_EN: track 0.00 -> 56.6 mm, vias 0 -> 2
- net /controller/SPI_NSS2: track 0.00 -> 50.0 mm, vias 0 -> 2
- net GND: track 449.4 -> 498.3 mm, vias 12 -> 77
- net /controller/SPI_NSS1: track 0.00 -> 45.1 mm, vias 0 -> 2
- net /controller/STIR_EN: track 0.00 -> 39.8 mm, vias 0 -> 4
- net +5V: track 197.8 -> 237.3 mm, vias 4 -> 9
- net /controller/AUX2: track 0.00 -> 35.8 mm, vias 0 -> 3
- net /controller/AUX1: track 0.00 -> 33.0 mm, vias 0 -> 3
- net /controller/SWCLK: track 9.08 -> 42.1 mm, vias 0 -> 5
- net /controller/FAN_EN: track 0.00 -> 32.7 mm, vias 0 -> 2
- net /controller/AUX3: track 0.00 -> 32.2 mm, vias 0 -> 3
- net /controller/BUZZER: track 0.00 -> 31.6 mm, vias 0 -> 2
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- added copper zone on B.Cu, net GND
- added copper zone on F.Cu, net GND
Other:
- board text added: "+"
- board text added: "-"
- board text added: "12V"
- board text added: "3V3"
- board text added: "5V"
- board text added: "AUX"
- board text added: "AUX0"
- board text added: "AUX1"
- board text added: "AUX2"
- board text added: "AUX3"
- board text added: "BOOT0"
- board text added: "FAN"
- board text added: "G"
- board text added: "GND"
- board text added: "HEATER"
- board text added: "LED"
- board text added: "NC"
- board text added: "PWM"
- board text added: "RELAY"
- board text added: "RESET"
- board text added: "RX"
- board text added: "SCL"
- board text added: "SDA"
- board text added: "STIR"
- board text added: "SWCLK"
- board text added: "SWDIO"
- board text added: "TACH"
- board text added: "TC"
- board text added: "THERMISTOR"
- board text added: "TX"
- board text added: "kelvin-kontroller v1.0"
