File: hardware/kelvin-kontroller.kicad_sch (KiCad schematic)
At the start: 59 parts, among them J12 USB_B_Micro, J13 Conn_01x04 Header, J14 Conn_01x02 Terminals, J15 Conn_01x07 Header, Q5 Q_NPN_BEC, Q6 Q_NPN_BEC, SW2 SW_Push, SW3 RotaryEncoder_Switch, U5 AMS1117-3.3, U6 ESP32-WROOM-32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

Commit message: Hardware revision v1.0
Parts:
- R22, R23, R24, R26: LCSC C25091 -> C25092
Changed lines of the file:
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@@
       (effects (font (size 1.27 1.27)) hide)
     )
-    (property "LCSC" "C25091" (id 4) (at 242.57 199.39 0)
+    (property "LCSC" "C25092" (id 4) (at 242.57 199.39 0)
       (effects (font (size 1.27 1.27)) hide)
     )
@@
       (effects (font (size 1.27 1.27)) hide)
     )
-    (property "LCSC" "C25091" (id 4) (at 234.95 201.93 0)
+    (property "LCSC" "C25092" (id 4) (at 234.95 201.93 0)
       (effects (font (size 1.27 1.27)) hide)
     )
@@
       (effects (font (size 1.27 1.27)) hide)
     )
-    (property "LCSC" "C25091" (id 4) (at 180.34 39.37 0)
+    (property "LCSC" "C25092" (id 4) (at 180.34 39.37 0)
       (effects (font (size 1.27 1.27)) hide)
     )
@@
       (effects (font (size 1.27 1.27)) hide)
     )
-    (property "LCSC" "C25091" (id 4) (at 160.02 41.91 0)
-      (effects (font (size 1.27 1.27)) hide)
-    )
+    (property "LCSC" "C25092" (id 4) (at 160.02 41.91 0)
+      (effects (font (size 1.27 1.27)) hide)
+    )
